Commit message: Migration to ros2 for lidar sensors

File: urdf/asus_xtion_pro.urdf.xacro (robot description, xacro)
@@ -112,5 +112,5 @@
           <cameraInfoTopicName>rgb/camera_info</cameraInfoTopicName>
           <depthImageCameraInfoTopicName>depth/camera_info</depthImageCameraInfoTopicName>
-          <frameName>${prefix}depth_optical_frame</frameName>
+          <frame_name>${prefix}depth_optical_frame</frame_name>
           <baseline>0.1</baseline>
           <distortion_k1>0.0</distortion_k1>

File: urdf/axis.urdf.xacro (robot description, xacro)
@@ -141,5 +141,5 @@
           <imageTopicName>image_raw</imageTopicName>
           <cameraInfoTopicName>camera_info</cameraInfoTopicName>
-          <frameName>/${prefix}_optical_frame_link</frameName>
+          <frame_name>/${prefix}_optical_frame_link</frame_name>
           <hackBaseline>0.0</hackBaseline>
           <distortionK1>0.0</distortionK1>

File: urdf/axis_m5013.urdf.xacro (robot description, xacro)
@@ -142,5 +142,5 @@
 					<imageTopicName>image_raw</imageTopicName>
 					<cameraInfoTopicName>camera_info</cameraInfoTopicName>
-					<frameName>${prefix}_optical_frame_link</frameName>
+					<frame_name>${prefix}_optical_frame_link</frame_name>
 					<!-- this is just which name the Image msg will have, it does not affect the simulation.
 					     However must be set to the optical_frame,  -->

File: urdf/axis_m5525.urdf.xacro (robot description, xacro)
@@ -144,5 +144,5 @@
 					<imageTopicName>image_raw</imageTopicName>
 					<cameraInfoTopicName>camera_info</cameraInfoTopicName>
-					<frameName>${prefix}_optical_frame_link</frameName>
+					<frame_name>${prefix}_optical_frame_link</frame_name>
 					<!-- this is just which name the Image msg will have, it does not affect the simulation.
 					     However must be set to the optical_frame,  -->

File: urdf/axis_q8641.urdf.xacro (robot description, xacro)
@@ -175,5 +175,5 @@
           <imageTopicName>image_raw</imageTopicName>
           <cameraInfoTopicName>camera_info</cameraInfoTopicName>
-          <frameName>/${prefix}_optical_frame_link</frameName>
+          <frame_name>/${prefix}_optical_frame_link</frame_name>
           <hackBaseline>0.0</hackBaseline>
           <distortionK1>0.0</distortionK1>

File: urdf/benewake_ce30.urdf.xacro (robot description, xacro)
@@ -81,5 +81,5 @@
           <plugin name="${prefix}_controller" filename="${plugin_lib}">
             <topicName>${prefix_topic}/points</topicName>
-            <frameName>/${prefix}_link</frameName>
+            <frame_name>/${prefix}_link</frame_name>
             <gaussianNoise>0.008</gaussianNoise>
           </plugin>

File: urdf/benewake_ce30d.urdf.xacro (robot description, xacro)
@@ -82,5 +82,5 @@
           <plugin name="${prefix}_controller" filename="${plugin_lib}">
             <topicName>${prefix_topic}/points</topicName>
-            <frameName>/${prefix}_link</frameName>
+            <frame_name>/${prefix}_link</frame_name>
             <gaussianNoise>0.008</gaussianNoise>
           </plugin>

File: urdf/embedded_s.urdf.xacro (robot description, xacro)
@@ -87,5 +87,5 @@
           <cameraInfoTopicName>rgb/camera_info</cameraInfoTopicName>
           <depthImageCameraInfoTopicName>depth/camera_info</depthImageCameraInfoTopicName>
-          <frameName>/${prefix}_depth_optical_frame</frameName>
+          <frame_name>/${prefix}_depth_optical_frame</frame_name>
           <baseline>0.1</baseline>
           <distortion_k1>0.0</distortion_k1>

File: urdf/fotonic_e.urdf.xacro (robot description, xacro)
@@ -89,5 +89,5 @@
           <depthImageCameraInfoTopicName>depth/camera_info</depthImageCameraInfoTopicName>
           <pointCloudTopicName>points</pointCloudTopicName>
-          <frameName>${prefix}_depth_optical_frame_link</frameName>
+          <frame_name>${prefix}_depth_optical_frame_link</frame_name>
           <pointCloudCutoff>0.5</pointCloudCutoff>
           <distortionK1>0</distortionK1>

File: urdf/hokuyo3d.urdf.xacro (robot description, xacro)
@@ -79,5 +79,5 @@
           <plugin name="${prefix}_controller" filename="${plugin_lib}">
                     <topicName>points</topicName>
-                    <frameName>${prefix}_link</frameName>
+                    <frame_name>${prefix}_link</frame_name>
                             <ignoreTfPrefix>1</ignoreTfPrefix>
                 </plugin>

File: urdf/hokuyo_urg04lx.urdf.xacro (robot description, xacro)
@@ -38,9 +38,9 @@
       <xacro:if value="${gpu}">
         <xacro:property name="ray_type" value="gpu_ray" />
-        <xacro:property name="plugin_lib" value="libgazebo_ros_gpu_laser.so" />
+        <xacro:property name="plugin_lib" value="libgazebo_ros_ray_sensor.so" />
       </xacro:if>
       <xacro:unless value="${gpu}">
         <xacro:property name="ray_type" value="ray" />
-        <xacro:property name="plugin_lib" value="libgazebo_ros_laser.so" />
+        <xacro:property name="plugin_lib" value="libgazebo_ros_ray_sensor.so" />
       </xacro:unless>
       <sensor type="${ray_type}" name="${prefix}_sensor">
@@ -69,6 +69,8 @@
         </ray>
         <plugin name="${prefix}_controller" filename="${plugin_lib}">
-          <topicName>${prefix_topic}/scan</topicName>
-          <frameName>${prefix}_link</frameName>
+          <ros>
+            <remapping>~/out:=${prefix_topic}/scan</remapping>
+          </ros>
+          <frame_name>${prefix}_link</frame_name>
           <ignoreTfPrefix>1</ignoreTfPrefix>
         </plugin>

File: urdf/hokuyo_ust10lx.urdf.xacro (robot description, xacro)
@@ -40,9 +40,9 @@
 			<xacro:if value="${gpu}">
         <xacro:property name="ray_type" value="gpu_ray" />
-        <xacro:property name="plugin_lib" value="libgazebo_ros_gpu_laser.so" />
+        <xacro:property name="plugin_lib" value="libgazebo_ros_ray_sensor.so" />
       </xacro:if>
       <xacro:unless value="${gpu}">
         <xacro:property name="ray_type" value="ray" />
-        <xacro:property name="plugin_lib" value="libgazebo_ros_laser.so" />
+        <xacro:property name="plugin_lib" value="libgazebo_ros_ray_sensor.so" />
       </xacro:unless>
 			<sensor type="${ray_type}" name="${prefix}_sensor">
@@ -73,6 +73,8 @@
 				</ray>
 				<plugin name="${prefix}_controller" filename="${plugin_lib}">
-					<topicName>${prefix_topic}/scan</topicName>
-					<frameName>/${prefix}_link</frameName>
+					<ros>
+            <remapping>~/out:=${prefix_topic}/scan</remapping>
+          </ros>
+					<frame_name>/${prefix}_link</frame_name>
 				</plugin>
 			</sensor>

File: urdf/hokuyo_ust20lx.urdf.xacro (robot description, xacro)
@@ -1,5 +1,5 @@
 <?xml version="1.0"?>
 <robot name="sensor_hokuyo_ust20lx" xmlns:xacro="http://wiki.ros.org/xacro">
-  <xacro:macro name="sensor_hokuyo_ust20lx" params="prefix parent prefix_topic:='front_laser' *origin min_angle:=-2.3562 max_angle:=2.3562 gpu:=^|true">
+  <xacro:macro name="sensor_hokuyo_ust20lx" params="prefix parent prefix_topic:='front_laser' *origin min_angle:=-2.3562 max_angle:=2.3562 gpu:=^|false">
 			<!--arg name="namespace" value="$(arg namespace)"/-->
     <joint name="${prefix}_base_joint" type="fixed">
@@ -41,13 +41,13 @@
 			<xacro:if value="${gpu}">
         <xacro:property name="ray_type" value="gpu_ray" />
-        <xacro:property name="plugin_lib" value="libgazebo_ros_gpu_laser.so" />
+        <xacro:property name="plugin_lib" value="libgazebo_ros_ray_sensor.so" />
       </xacro:if>
       <xacro:unless value="${gpu}">
         <xacro:property name="ray_type" value="ray" />
-        <xacro:property name="plugin_lib" value="libgazebo_ros_laser.so" />
+        <xacro:property name="plugin_lib" value="libgazebo_ros_ray_sensor.so" />
       </xacro:unless>
 			<sensor type="${ray_type}" name="${prefix}_sensor">
 				<pose>0 0 0 0 0 0</pose>
-				<visualize>false</visualize>
+				<visualize>true</visualize>
 				<update_rate>40</update_rate>
 				<ray>
@@ -74,6 +74,9 @@
 				</ray>
 				<plugin name="${prefix}_controller" filename="${plugin_lib}">
-					<topicName>${prefix_topic}/scan</topicName>
-					<frameName>/${prefix}_link</frameName>
+					<ros>
+            <remapping>~/out:=${prefix_topic}/scan</remapping>
+          </ros>
+					<frame_name>${prefix}_link</frame_name>
+          <output_type>sensor_msgs/LaserScan</output_type>
 				</plugin>
 			</sensor>

File: urdf/hokuyo_utm30lx.urdf.xacro (robot description, xacro)
@@ -38,9 +38,9 @@
 			<xacro:if value="${gpu}">
         <xacro:property name="ray_type" value="gpu_ray" />
-        <xacro:property name="plugin_lib" value="libgazebo_ros_gpu_laser.so" />
+        <xacro:property name="plugin_lib" value="libgazebo_ros_ray_sensor.so" />
       </xacro:if>
       <xacro:unless value="${gpu}">
         <xacro:property name="ray_type" value="ray" />
-        <xacro:property name="plugin_lib" value="libgazebo_ros_laser.so" />
+        <xacro:property name="plugin_lib" value="libgazebo_ros_ray_sensor.so" />
       </xacro:unless>
 			<sensor type="${ray_type}" name="${prefix}_sensor">
@@ -69,6 +69,8 @@
 				</ray>
 				<plugin name="${prefix}_controller" filename="${plugin_lib}">
-					<topicName>${prefix_topic}/scan</topicName>
-					<frameName>/${prefix}_link</frameName>
+					<ros>
+            <remapping>~/out:=${prefix_topic}/scan</remapping>
+          </ros>
+					<frame_name>/${prefix}_link</frame_name>
 				</plugin>
 			</sensor>

File: urdf/imu.urdf.xacro (robot description, xacro)
@@ -51,5 +51,5 @@
         <xyzOffset>0 0 0</xyzOffset>
         <rpyOffset>0 0 0</rpyOffset>
-		<frameName>${prefix}_link</frameName>
+		<frame_name>${prefix}_link</frame_name>
       </plugin>
       <pose>0 0 0 0 0 0</pose>

File: urdf/rplidar.urdf.xacro (robot description, xacro)
@@ -39,9 +39,9 @@
 			<xacro:if value="${gpu}">
         <xacro:property name="ray_type" value="gpu_ray" />
-        <xacro:property name="plugin_lib" value="libgazebo_ros_gpu_laser.so" />
+        <xacro:property name="plugin_lib" value="libgazebo_ros_ray_sensor.so" />
       </xacro:if>
       <xacro:unless value="${gpu}">
         <xacro:property name="ray_type" value="ray" />
-        <xacro:property name="plugin_lib" value="libgazebo_ros_laser.so" />
+        <xacro:property name="plugin_lib" value="libgazebo_ros_ray_sensor.so" />
       </xacro:unless>
 			<sensor type="${ray_type}" name="${prefix}_rplidar_sensor">
@@ -70,6 +70,8 @@
 				</ray>
 				<plugin name="${prefix}_controller" filename="${plugin_lib}">
-					<topicName>${prefix_topic}/scan</topicName>
-					<frameName>/${prefix}_laser_link</frameName>
+					<ros>
+            <remapping>~/out:=${prefix_topic}/scan</remapping>
+          </ros>
+					<frame_name>/${prefix}_laser_link</frame_name>
 				</plugin>
 			</sensor>

File: urdf/rplidar_a2.urdf.xacro (robot description, xacro)
@@ -39,9 +39,9 @@
 			<xacro:if value="${gpu}">
         <xacro:property name="ray_type" value="gpu_ray" />
-        <xacro:property name="plugin_lib" value="libgazebo_ros_gpu_laser.so" />
+        <xacro:property name="plugin_lib" value="libgazebo_ros_ray_sensor.so" />
       </xacro:if>
       <xacro:unless value="${gpu}">
         <xacro:property name="ray_type" value="ray" />
-        <xacro:property name="plugin_lib" value="libgazebo_ros_laser.so" />
+        <xacro:property name="plugin_lib" value="libgazebo_ros_ray_sensor.so" />
       </xacro:unless>
 			<sensor type="${ray_type}" name="${prefix}_rplidar_a2_sensor">
@@ -70,6 +70,8 @@
 				</ray>
 				<plugin name="${prefix}_controller" filename="${plugin_lib}">
-					<topicName>${prefix_topic}/scan</topicName>
-					<frameName>/${prefix}_link</frameName>
+					<ros>
+            <remapping>~/out:=${prefix_topic}/scan</remapping>
+          </ros>
+					<frame_name>/${prefix}_link</frame_name>
 				</plugin>
 			</sensor>

File: urdf/rs_bpearl.urdf.xacro (robot description, xacro)
@@ -98,5 +98,5 @@
           <plugin name="${prefix}_controller" filename="${plugin_lib}">
             <topicName>${prefix_topic}/points</topicName>
-            <frameName>/${prefix}_link</frameName>
+            <frame_name>/${prefix}_link</frame_name>
             <gaussianNoise>0.008</gaussianNoise>
           </plugin>

File: urdf/rslidar.urdf.xacro (robot description, xacro)
@@ -80,5 +80,5 @@
           <plugin name="${prefix}_controller" filename="${plugin_lib}">
             <topicName>${prefix_topic}/points</topicName>
-            <frameName>/${prefix}_link</frameName>
+            <frame_name>/${prefix}_link</frame_name>
             <gaussianNoise>0.008</gaussianNoise>
           </plugin>

File: urdf/rslidar_mems.urdf.xacro (robot description, xacro)
@@ -84,5 +84,5 @@
           <plugin name="${prefix}_controller" filename="${plugin_lib}">
               <topicName>/robot/front_3d_laser/point_cloud</topicName>
-              <frameName>/${prefix}_link</frameName>
+              <frame_name>/${prefix}_link</frame_name>
               <ignoreTfPrefix>1</ignoreTfPrefix>
           </plugin>
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