Commit message: gpu=false because gpu_ray cant detect actor

File: urdf/sick_nanoscan3.urdf.xacro (robot description, xacro)
@@ -2,5 +2,5 @@
 <robot name="sensor_sick_nanoscan3"
 	xmlns:xacro="http://wiki.ros.org/xacro">
-	<xacro:macro name="sensor_sick_nanoscan3" params="prefix parent prefix_topic:='front_laser' *origin max_angle:=2.3998 min_angle:=-2.3998 gpu:=^|true">
+	<xacro:macro name="sensor_sick_nanoscan3" params="prefix parent prefix_topic:='front_laser' *origin max_angle:=2.3998 min_angle:=-2.3998 gpu:=^|false">
 		<joint name="${prefix}_base_joint" type="fixed">
 			<xacro:insert_block name="origin" />

Commit message: Using gpu ray for back laser to fix inconsistent ray spectrum. Surprisingly, gpu ray can detect actor on my private desktop computer.

File: urdf/sick_nanoscan3.urdf.xacro (robot description, xacro)
@@ -2,5 +2,5 @@
 <robot name="sensor_sick_nanoscan3"
 	xmlns:xacro="http://wiki.ros.org/xacro">
-	<xacro:macro name="sensor_sick_nanoscan3" params="prefix parent prefix_topic:='front_laser' *origin max_angle:=2.3998 min_angle:=-2.3998 gpu:=^|false">
+	<xacro:macro name="sensor_sick_nanoscan3" params="prefix parent prefix_topic:='front_laser' *origin max_angle:=2.3998 min_angle:=-2.3998 gpu:=^|true">
 		<joint name="${prefix}_base_joint" type="fixed">
 			<xacro:insert_block name="origin" />
@@ -50,5 +50,5 @@
 			<sensor type="${ray_type}" name="${prefix}_sensor">
 				<pose>0 0 0 0 0 0</pose>
-				<visualize>false</visualize>
+				<visualize>true</visualize>
 				<update_rate>12.5</update_rate>
 				<ray>

Commit message: gpu=false and visualize=false for nanoscan3

File: urdf/sick_nanoscan3.urdf.xacro (robot description, xacro)
@@ -2,5 +2,5 @@
 <robot name="sensor_sick_nanoscan3"
 	xmlns:xacro="http://wiki.ros.org/xacro">
-	<xacro:macro name="sensor_sick_nanoscan3" params="prefix parent prefix_topic:='front_laser' *origin max_angle:=2.3998 min_angle:=-2.3998 gpu:=^|true">
+	<xacro:macro name="sensor_sick_nanoscan3" params="prefix parent prefix_topic:='front_laser' *origin max_angle:=2.3998 min_angle:=-2.3998 gpu:=^|false">
 		<joint name="${prefix}_base_joint" type="fixed">
 			<xacro:insert_block name="origin" />
@@ -50,5 +50,5 @@
 			<sensor type="${ray_type}" name="${prefix}_sensor">
 				<pose>0 0 0 0 0 0</pose>
-				<visualize>true</visualize>
+				<visualize>false</visualize>
 				<update_rate>12.5</update_rate>
 				<ray>
