Commit message: Small adjustments to rs_lidar_16

File: urdf/rs_lidar_16.urdf.xacro (robot description, xacro)
@@ -2,5 +2,5 @@
 <robot name="sensor_rs_lidar_16"
 	xmlns:xacro="http://wiki.ros.org/xacro">
-	<xacro:macro name="sensor_rs_lidar_16" params="prefix parent prefix_topic:='front_laser' *origin max_angle:=2.3562 min_angle:=-2.3562 gpu:=^|false">
+	<xacro:macro name="sensor_rs_lidar_16" params="prefix parent prefix_topic:='top_laser' *origin max_angle:=2.3562 min_angle:=-2.3562 gpu:=^|false">
 		<joint name="${prefix}_base_joint" type="fixed">
 			<xacro:insert_block name="origin" />
@@ -62,6 +62,6 @@
                                                         <samples>16</samples>
                                                         <resolution>1</resolution>
-                                                        <min_angle>-0.261799</min_angle>
-                                                        <max_angle>0.261799</max_angle>
+                                                        <min_angle>-0.261799</min_angle> <!-- -15° -->
+                                                        <max_angle>0.261799</max_angle> <!-- +15° -->
                                                 </vertical>
                                         </scan>
@@ -79,5 +79,5 @@
                                 <plugin name='${prefix}_controller' filename="${plugin_lib}">
                                         <ros>
-                                                <remapping>~/out:=${prefix_topic}/robosense_scan</remapping>
+                                                <remapping>~/out:=${prefix_topic}/points</remapping>
                                         </ros>
                                         <frame_name>${prefix}_link</frame_name>
