Commit message: xacro anpassung realsense

File: urdf/intel_r430.urdf.xacro (robot description, xacro)
@@ -102,8 +102,8 @@
     </joint>
     <link name="${prefix}_camera_fisheye_optical_frame"/>
+  </xacro:macro>
   <!-- RGBD sensor for simulation, same as Kinect -->
   <sensor_r430_gazebo/>
-  </xacro:macro>
-   <xacro:macro name="sensor_r430_gazebo">
+  <xacro:macro name="sensor_r430_gazebo">
     <!-- gazebo reference="${prefix}_rgb_base_link" -->
     <gazebo reference="${prefix}_camera_link">
@@ -168,9 +168,9 @@
             -->
             <ros>
-              <argument>image_raw:=custom_image</argument>
-              <argument>image_depth:=custom_image_depth</argument>
-              <argument>camera_info:=custom_info_raw</argument>
-              <argument>camera_info_depth:=custom_info_depth</argument>
-              <argument>points:=custom_points</argument>
+              <xacro:argument>image_raw:=custom_image</xacro:argument>
+              <xacro:argument>image_depth:=custom_image_depth</xacro:argument>
+              <xacro:argument>camera_info:=custom_info_raw</xacro:argument>
+              <xacro:argument>camera_info_depth:=custom_info_depth</xacro:argument>
+              <xacro:argument>points:=custom_points</xacro:argument>
             </ros>
             <!-- Set camera name. If empty, defaults to sensor name (i.e. "sensor_name") -->

File: urdf/ueye_cp_gige.urdf.xacro (robot description, xacro)
@@ -3,5 +3,5 @@
   <xacro:macro name="sensor_ueye_cp_gige" params="prefix parent *origin">
     <joint name="${prefix}_joint" type="fixed">
-      <insert_block name="origin"/>
+      <xacro:insert_block name="origin"/>
       <parent link="${parent}"/>
       <child link="${prefix}_base_link"/>
