Commit message: rs_bpaerl update to new plugin

File: urdf/rs_bpearl.urdf.xacro (robot description, xacro)
@@ -63,9 +63,9 @@
         <!-- Using GPU needs: https://github.com/RobotnikAutomation/velodyne_simulator -->
         <xacro:property name="ray_type" value="gpu_ray" />
-        <xacro:property name="plugin_lib" value="libgazebo_ros_velodyne_gpu_laser.so" />
+        <xacro:property name="plugin_lib" value="libGazeboRosVelodyneLaser.so" />
       </xacro:if>
       <xacro:unless value="${gpu}">
         <xacro:property name="ray_type" value="ray" />
-        <xacro:property name="plugin_lib" value="libgazebo_ros_velodyne_laser.so" />
+        <xacro:property name="plugin_lib" value="libGazeboRosVelodyneLaser.so" />
       </xacro:unless>
         <sensor type="${ray_type}" name="${prefix}_sensor">
